File: hardware/logic/RATT_REV0.sch (EAGLE design)
At the start: 132 parts, among them IC1 TLP292-4, IC13 MCP73831, IC16 PCA9539PW, IC2 CPC1002N, IC3 CPC1002N, IC4 CPC1002N, IC5 CPC1002N, J1 4P-2.0, J2 4P-2.0, J3 F-1X06-SIP-100-40, J4 4P-2.0, J6 4P-2.0, J7 PHOENIX1803484, J8 PHOENIX1803484, Q1 2.5A/30V, Q2 MBT3904DW1T1, Q3 2.5A/30V, Q5 2N7002, Q6 2.5A/30V, U1 RPI-ZERO, U5 AP2112K-3.3V

Commit message: Just need to do the dumb power path
I forget what I did, but it wasn't the power path yet
Parts:
- removed C2: 10uF, SparkFun-Capacitors:CAP0805
- removed C21: 0.1uF, MakeItLabs:CAP0603
- removed D1: Yellow, SparkFun-LED:LED-YELLOW0603
- removed D4: BAT20J, SparkFun-DiscreteSemi:DIODE-SCHOTTKY-BAT20J
- removed F1: 500mA, SparkFun-PowerIC:PTCSMD
- removed J3: F-1X06-SIP-100-40, con-headers-jp:F-1X06-SIP-100-40
- removed SJ2: JUMPER-PAD-2-NC_BY_TRACE, SparkFun-Passives:JUMPER-PAD-2-NC_BY_TRACE
- added J5: F-1X04-SIP-100-40, con-headers-jp:F-1X04-SIP-100-40
- added LED4, LED5, LED6: RED, SparkFun-LED:LED-RED0603
- added R56, R57: 1K, SparkFun-Resistors:1KOHM-1/10W-1%(0603)
- added R58: 1k, SparkFun-Resistors:10KOHM-0603-1/10W-1%
- added R59: 10k, SparkFun-Resistors:10KOHM-0603-1/10W-1%
- IC13: value MCP73831 -> MCP73832
- R24: value 10k -> 1k
- renumbered X2 to J100
Connections:
- removed net 3.3REG_EN: D4.A
- removed net VUSB-RAW: F1.1
- removed net V_USB: F1.2, FB3.P$2
- new net N$53: Q2Q1.B, R58.1
- net +3V3: now also R59.2
- net +5V: now also FB3.P$2, R56.1, R58.2
- net 3.3V: now also R21.1; no longer SJ2.2
- net 5V_RFID_TX: now also J5.3; no longer J3.6
- net CHARGE_STATUS: now also LED6.C, U1.GPIO12; no longer D1.C
- net GND: now also J5.1, LED4.C, LED5.C, Q2Q1.E; no longer C2.2, C21.2, J3.1
- net N$12: now also LED5.A, R57.2; no longer R21.1, SJ2.1
- net N$17: now also LED6.A; no longer D1.A
- net N$18: no longer D4.C
- net N$50: now also LED4.A, R56.2; no longer C2.1, C21.1, FB4.P$1, J3.3
- net N$51: now also FB4.P$1, J5.2; no longer J3.2
- net PWR_LOSS: now also Q2Q1.C, R59.1
- net RFID_RX: now also J5.4, U1.TXD0/GPIO14; no longer J3.5, U1.RXD0/GPIO15
- net RFID_TX: now also U1.RXD0/GPIO15; no longer U1.TXD0/GPIO14
- net VIN: now also R57.1
Other:
- note added: "3.3V is supplied by this circuit or by the Pi Module"
- note added: "LCD"
- note added: "Pi Supplies 3.3V"
- note removed: "LCD Options"
- note removed: "SJ2 disconnects the power LED (for power saving)."
- moved on the sheet: C1, C10, C19, C25, C7, C8, FB3, FB4, IC13, JP2, LED3, Q2Q1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

Commit message: Renamed Power Supply Nets
+5VIN = Input from Dc brick
+5VB = 5V or Battery backed supply
+3.3V = +3.3V supply created from +5VB by either Pi or reg circuit
Parts:
- removed SJ1: JUMPER-PAD-2-NC_BY_TRACE, SparkFun-Passives:JUMPER-PAD-2-NC_BY_TRACE
Connections:
- removed net +3V3: C18.1, C20.1, C22.1, C23.1, FB4.P$2, IC16.VCC, JP1.8, R1.2, R13.2, R2.2, R25.2, R28.2, R29.2, R3.2, R30.2, R31.2, R32.2, R33.2, R34.2, R4.2, R41.2, R42.2, R5.2, R55.2, R59.2, SJ4.2
- removed net +5V: C19.1, D10.C2, D2.C2, D3.C2, D5.C2, D6.C2, D7.C2, D8.C2, D9.C2, FB3.P$2, IC13.VIN, J1.3, J100.1, J2.3, J4.3, J6.3, JP1.4, Q1.G, Q6.D, R17.2, R18.1, R56.1, R58.2, R9.2
- removed net 3.3V: C10.1, R21.1, R36.1, U5.OUT
- removed net N$16: R19.2, SJ1.1
- removed net VIN: C17.1, C7.1, C9.1, Q1.S, Q6.S, R10.1, R24.2, R57.1, R7.2, R8.2, U1.5V0@1, U1.5V0@2, U2.VDD, U5.IN
- new net +3.3V: C10.1, C18.1, C20.1, C22.1, C23.1, FB4.P$2, IC16.VCC, JP1.8, R1.2, R13.2, R2.2, R21.1, R25.2, R28.2, R29.2, R3.2, R30.2, R31.2, R32.2, R33.2, R34.2, R36.1, R4.2, R41.2, R42.2, R5.2, R55.2, R59.2, SJ4.2, U5.OUT
- new net +5VB: C17.1, C7.1, C9.1, D10.C2, D2.C2, D3.C2, D5.C2, D6.C2, D7.C2, D8.C2, D9.C2, FB3.P$2, Q1.S, Q6.S, R10.1, R24.2, R57.1, R7.2, R8.2, U1.5V0@1, U1.5V0@2, U2.VDD, U5.IN
- new net +5VIN: C19.1, IC13.VIN, J1.3, J100.1, J2.3, J4.3, J6.3, JP1.4, Q1.G, Q6.D, R17.2, R18.1, R56.1, R58.2, R9.2
- net N$14: now also R19.2; no longer SJ1.2
Other:
- note removed: "SJ1 can be cut to modify the charge- current programming resistor."
- moved on the sheet: C19, C8, IC13, JP2, LED6, R18, R19, R36

Commit message: Schematic Done! (ref des and attributes may change)
Initial pass on schematic done.  Ref Des and attributes will change before it is finished though
Parts:
- removed Q1, Q3, Q6: 2.5A/30V, SparkFun-DiscreteSemi:MOSFET-PCHANNELDMG2307L
- removed Q2: MBT3904DW1T1, esp32-thing-temp:MBT3904DW1T1
- removed Q4, Q7: (no value), DURRIDGE-TRANSISTORS:TRANSISTOR_NPNSOT23-3
- removed R10, R17, R59: 10k, SparkFun-Resistors:10KOHM-0603-1/10W-1%
- removed R58, R9: 1k, SparkFun-Resistors:10KOHM-0603-1/10W-1%
- removed U2: (no value), Adafruit_MAX98357:AUDIOAMP_MAX98357
- removed X1: (no value), Adafruit_MAX98357:TERMBLOCK_1X2
- added C2, C3: 0.1uF, SparkFun-Capacitors:CAP0603-CAP
- added IC200: TPS2115AIPWRQ1, Texas Instruments_By_element14_Batch_1:TPS2115AIPWRQ1
- added IC300: MAx98357, Adafruit_MAX98357:AUDIOAMP_MAX98357
- added J200: (no value), Adafruit_MAX98357:TERMBLOCK_1X2
- added R60: 1k, SparkFun-Resistors:10KOHM-0603-1/10W-1%
- added R61: 10k, SparkFun-Resistors:10KOHM-0603-1/10W-1%
- R12: value 1k -> 10k
Connections:
- removed net !SHUTDOWN: R12.1, U1.GPIO27/GEN2
- removed net N$10: Q1.D, Q3.D
- removed net N$35: Q7.B, R9.1
- removed net N$38: Q4.B, R12.2
- removed net N$53: Q2Q1.B, R58.1
- removed net N$9: Q6.G, Q7.C, R10.2
- removed net PWR_LOSS: Q2Q1.C, R59.1, U1.GPIO26
- new net !PWR_LOSS: IC200.STAT, R61.1, U1.GPIO26
- new net SHUTDOWN: IC200.D1, R12.2, U1.GPIO27/GEN2
- net +3.3V: now also R61.2; no longer R59.2
- net +5VB: now also IC200.D0, IC200.OUT, IC300.VDD, R11.2; no longer Q1.S, Q6.S, R10.1, U2.VDD
- net +5VIN: now also C3.1, IC200.IN2; no longer Q1.G, Q6.D, R17.2, R58.2, R9.2
- net GND: now also C2.2, C3.2, IC200.GND, IC300.GND, R11.1, R12.1, R60.1; no longer Q2Q1.E, Q4.E, Q7.E, R17.1, U2.GND
- net I2S_BCK: now also IC300.BCLK; no longer U2.BCLK
- net I2S_DOUT: now also IC300.DIN; no longer U2.DIN
- net I2S_WS/LRCLK: now also IC300.LRCLK; no longer U2.LRCLK
- net N$1: now also IC300.GAIN; no longer U2.GAIN
- net N$2: now also IC300.OUTP; no longer U2.OUTP
- net N$37: now also IC200.ILIM, R60.2; no longer Q3.G, Q4.C, R11.1
- net N$4: now also IC300.OUTN; no longer U2.OUTN
- net N$5: now also IC300.!SD_MODE; no longer U2.!SD_MODE
- net N$6: now also J200.1; no longer X1.1
- net N$7: now also J200.2; no longer X1.2
- net V_BATT: now also C2.1, IC200.IN1; no longer Q3.S, R11.2
Other:
- note added: "3.3V LDO"
- note added: "D1 D0 IN2>IN1 STAT OUT 0 0 X HI-Z IN2 0 1 NO 0 IN1 0 1 YES HI-Z IN2 1 0 X 0 IN1 1 1 X 0 HI-Z"
- note added: "IO Systems"
- note added: "MakeIt Labs RATT"
- note added: "Not Used"
- note added: "Power LEDs"
- note added: "Power Source Switch"
- note added: "Power Systems"
- note added: "RATT"
- note removed: "TODO: Revise power path circuit"
- moved on the sheet: C1, C10, C17, C19, C22, C23, C25, C5, C6, C7, C8, C9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

Commit message: Moved all parts into MakeItLabs Library
Parts:
- removed U5: AP2112K-3.3V, SparkFun-PowerIC:V_REG_LDOSMD
- added IC500: AP2112K-3.3V, MakeItLabs:V_REG_LDOSMD
- C1, C20, C23: device SparkFun-Capacitors:CAP0805 -> MakeItLabs:CAP0805
- C10: device SparkFun-Capacitors:2.2UF-0603-10V-20% -> MakeItLabs:CAP0603
- C18, C2, C22, C3: device SparkFun-Capacitors:CAP0603-CAP -> MakeItLabs:CAP0603
- C19, C8: device SparkFun-Capacitors:4.7UF0603 -> MakeItLabs:CAP0603
- C7: device SparkFun-Capacitors:1.0UF-0805-25V-(+80/-20%) -> MakeItLabs:CAP0603
- D10, D2, D3, D5, D6, D7, D8, D9: device DURRIDGE-DIODES:BAT54S -> MakeItLabs:BAT54S
- FB1, FB2: device Adafruit_MAX98357:FERRITE -> MakeItLabs:FERRITE
- FB3, FB4: device DURRIDGE-INDUCTORS:FERRITE -> MakeItLabs:FERRITE
- IC1: device DURRIDGE-IC:TLP292-4 -> MakeItLabs:TLP292-4
- IC13: device SparkFun-PowerIC:MCP73831 -> MakeItLabs:MCP73831
- IC16: device Texas Instruments_By_element14_Batch_1:PCA9539PW -> MakeItLabs:PCA9539PW
- IC200: device Texas Instruments_By_element14_Batch_1:TPS2115AIPWRQ1 -> MakeItLabs:TPS2115AIPWRQ1
- IC300: value MAx98357 -> MAX98357; device Adafruit_MAX98357:AUDIOAMP_MAX98357 -> MakeItLabs:AUDIOAMP_MAX98357
- J100, J200: device Adafruit_MAX98357:TERMBLOCK_1X2 -> MakeItLabs:TERMBLOCK_1X2
- J5: device con-headers-jp:F-1X04-SIP-100-40 -> MakeItLabs:F-1X04-SIP-100-40
- JP1: device pinhead:PINHD-2X8 -> MakeItLabs:PINHD-2X8
- JP2: device SparkFun-Connectors:M02JST-PTH-2 -> MakeItLabs:M02JST-PTH-2
- LED1, LED2: device SparkFun-LED:LED5MM -> MakeItLabs:LED5MM
- LED3, LED4, LED5, LED6: device SparkFun-LED:LED-RED0603 -> MakeItLabs:LED-RED0603
- Q5: device zetex:NMOSSOT23 -> MakeItLabs:NMOSSOT23
- R1: device SparkFun-Passives:RESISTOR0603-RES -> MakeItLabs:RESISTOR0603
- R11, R12, R24, R60, R61: device SparkFun-Resistors:10KOHM-0603-1/10W-1% -> MakeItLabs:RESISTOR0603
- R14, R15, R16, R22: device DURRIDGE-RESISTORS:RESISTOR2512 -> MakeItLabs:RESISTOR2512
- R18, R21, R36, R56, R57: device SparkFun-Resistors:1KOHM-1/10W-1%(0603) -> MakeItLabs:RESISTOR0603
- R19: device SparkFun-Resistors:2.0KOHM1/10W5%(0603) -> MakeItLabs:RESISTOR0603
- SW0, SW1, SW2, SW3: device MakeIt_Labs:ESWITCH_320 -> MakeItLabs:ESWITCH_320
- U1: device RPI-Zero:RPI-ZERO -> MakeItLabs:RPI-ZERO
Connections:
- net +3.3V: now also IC500.OUT; no longer U5.OUT
- net +5VB: now also IC500.IN; no longer U5.IN
- net GND: now also IC500.GND; no longer U5.GND
- net N$18: now also IC500.EN; no longer U5.EN

Commit message: most stuff placed
Parts:
- renumbered U1 to J87
Changed lines of the file:
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@@
 <setting verticaltext="up"/>
 </settings>
-<grid distance="0.1" unitdist="inch" unit="inch" style="lines" multiple="1" display="yes" altdistance="0.01" altunitdist="inch" altunit="inch"/>
+<grid distance="0.1" unitdist="inch" unit="inch" style="lines" multiple="1" display="no" altdistance="0.01" altunitdist="inch" altunit="inch"/>
 <layers>
 <layer number="1" name="Top" color="4" fill="1" visible="no" active="no"/>
@@
 <part name="SUPPLY28" library="MakeItLabs" deviceset="GND" device=""/>
 <part name="R35" library="MakeItLabs" deviceset="RESISTOR" device="0603" value="10K"/>
-<part name="U1" library="MakeItLabs" deviceset="RPI-ZERO" device=""/>
+<part name="J87" library="MakeItLabs" deviceset="RPI-ZERO" device=""/>
 <part name="R36" library="MakeItLabs" deviceset="RESISTOR" device="0603" value="1K"/>
 <part name="SUPPLY9" library="MakeItLabs" deviceset="GND" device=""/>
@@
 <attribute name="VALUE" x="53.34" y="83.82" size="1.27" layer="96" font="vector" rot="R180"/>
 </instance>
-<instance part="U1" gate="G$1" x="60.96" y="200.66"/>
+<instance part="J87" gate="G$1" x="60.96" y="200.66"/>
 <instance part="R36" gate="G$1" x="269.24" y="218.44" rot="MR270"/>
 <instance part="SUPPLY9" gate="GND" x="88.9" y="177.8" smashed="yes">
@@
 </segment>
 <segment>
-<pinref part="U1" gate="G$1" pin="GPIO2/SDA1"/>
+<pinref part="J87" gate="G$1" pin="GPIO2/SDA1"/>
 <wire x1="38.1" y1="228.6" x2="33.02" y2="228.6" width="0.1524" layer="91"/>
 <label x="33.02" y="228.6" size="1.27" layer="95" rot="R180" xref="yes"/>
@@
 </segment>
 <segment>
-<pinref part="U1" gate="G$1" pin="GPIO3/SCL1"/>
+<pinref part="J87" gate="G$1" pin="GPIO3/SCL1"/>
 <wire x1="38.1" y1="226.06" x2="33.02" y2="226.06" width="0.1524" layer="91"/>
 <label x="33.02" y="226.06" size="1.27" layer="95" rot="R180" xref="yes"/>
@@
 <wire x1="86.36" y1="203.2" x2="91.44" y2="203.2" width="0.1524" layer="91"/>
 <label x="91.44" y="203.2" size="1.27" layer="95" xref="yes"/>
-<pinref part="U1" gate="G$1" pin="!CE0!/GPIO8"/>
+<pinref part="J87" gate="G$1" pin="!CE0!/GPIO8"/>
 </segment>
 </net>
@@
 <wire x1="38.1" y1="203.2" x2="33.02" y2="203.2" width="0.1524" layer="91"/>
 <label x="33.02" y="203.2" size="1.27" layer="95" rot="R180" xref="yes"/>
-<pinref part="U1" gate="G$1" pin="GPIO11/SCLK"/>
+<pinref part="J87" gate="G$1" pin="GPIO11/SCLK"/>
 </segment>
 </net>
@@
 <wire x1="38.1" y1="205.74" x2="33.02" y2="205.74" width="0.1524" layer="91"/>
 <label x="33.02" y="205.74" size="1.27" layer="95" rot="R180" xref="yes"/>
-<pinref part="U1" gate="G$1" pin="GPIO9/MISO"/>
+<pinref part="J87" gate="G$1" pin="GPIO9/MISO"/>
 </segment>
 </net>
@@
 <wire x1="38.1" y1="208.28" x2="33.02" y2="208.28" width="0.1524" layer="91"/>
 <label x="33.02" y="208.28" size="1.27" layer="95" rot="R180" xref="yes"/>
-<pinref part="U1" gate="G$1" pin="GPIO10/MOSI"/>
+<pinref part="J87" gate="G$1" pin="GPIO10/MOSI"/>
 </segment>
 </net>
@@
 </segment>
 <segment>
-<pinref part="U1" gate="G$1" pin="GPIO5"/>
+<pinref part="J87" gate="G$1" pin="GPIO5"/>
 <wire x1="38.1" y1="195.58" x2="33.02" y2="195.58" width="0.1524" layer="91"/>
 <label x="33.02" y="195.58" size="1.27" layer="95" rot="R180" xref="yes"/>
@@
 <wire x1="86.36" y1="210.82" x2="91.44" y2="210.82" width="0.1524" layer="91"/>
 <label x="91.44" y="210.82" size="1.27" layer="95" font="vector" xref="yes"/>
-<pinref part="U1" gate="G$1" pin="GEN5/GPIO24"/>
+<pinref part="J87" gate="G$1" pin="GEN5/GPIO24"/>
 </segment>
 </net>
@@
 <wire x1="86.36" y1="213.36" x2="91.44" y2="213.36" width="0.1524" layer="91"/>
 <label x="91.44" y="213.36" size="1.27" layer="95" font="vector" xref="yes"/>
-<pinref part="U1" gate="G$1" pin="GEN4/GPIO23"/>
+<pinref part="J87" gate="G$1" pin="GEN4/GPIO23"/>
 </segment>
 </net>
@@
 <wire x1="38.1" y1="187.96" x2="33.02" y2="187.96" width="0.1524" layer="91"/>
 <label x="33.02" y="187.96" size="1.27" layer="95" font="vector" rot="R180" xref="yes"/>
-<pinref part="U1" gate="G$1" pin="GPIO19"/>
+<pinref part="J87" gate="G$1" pin="GPIO19"/>
 </segment>
 </net>
@@
 <wire x1="86.36" y1="218.44" x2="91.44" y2="218.44" width="0.1524" layer="91"/>
 <label x="91.44" y="218.44" size="1.27" layer="95" font="vector" xref="yes"/>
-<pinref part="U1" gate="G$1" pin="GPIO18"/>
+<pinref part="J87" gate="G$1" pin="GPIO18"/>
 </segment>
 </net>
@@
 <wire x1="86.36" y1="182.88" x2="91.44" y2="182.88" width="0.1524" layer="91"/>
 <label x="91.44" y="182.88" size="1.27" layer="95" font="vector" xref="yes"/>
-<pinref part="U1" gate="G$1" pin="GPIO21"/>
+<pinref part="J87" gate="G$1" pin="GPIO21"/>
 </segment>
 </net>
@@
 </segment>
 <segment>
-<pinref part="U1" gate="G$1" pin="GND@3"/>
+<pinref part="J87" gate="G$1" pin="GND@3"/>
 <pinref part="SUPPLY10" gate="GND" pin="GND"/>
 <wire x1="38.1" y1="182.88" x2="35.56" y2="182.88" width="0.1524" layer="91"/>
@@
 <wire x1="35.56" y1="182.88" x2="35.56" y2="200.66" width="0.1524" layer="91"/>
 <junction x="35.56" y="182.88"/>
-<pinref part="U1" gate="G$1" pin="GND@2"/>
+<pinref part="J87" gate="G$1" pin="GND@2"/>
 <wire x1="35.56" y1="200.66" x2="38.1" y2="200.66" width="0.1524" layer="91"/>
 <wire x1="35.56" y1="200.66" x2="35.56" y2="220.98" width="0.1524" layer="91"/>
 <junction x="35.56" y="200.66"/>
-<pinref part="U1" gate="G$1" pin="GND@1"/>
+<pinref part="J87" gate="G$1" pin="GND@1"/>
 <wire x1="35.56" y1="220.98" x2="38.1" y2="220.98" width="0.1524" layer="91"/>
 </segment>
@@
 <pinref part="SUPPLY9" gate="GND" pin="GND"/>
 <wire x1="88.9" y1="180.34" x2="88.9" y2="190.5" width="0.1524" layer="91"/>
-<pinref part="U1" gate="G$1" pin="GND@8"/>
+<pinref part="J87" gate="G$1" pin="GND@8"/>
 <wire x1="88.9" y1="190.5" x2="88.9" y2="195.58" width="0.1524" layer="91"/>
 <wire x1="88.9" y1="195.58" x2="88.9" y2="208.28" width="0.1524" layer="91"/>
@@
 <wire x1="88.9" y1="215.9" x2="88.9" y2="226.06" width="0.1524" layer="91"/>
 <wire x1="88.9" y1="226.06" x2="86.36" y2="226.06" width="0.1524" layer="91"/>
-<pinref part="U1" gate="G$1" pin="GND@7"/>
+<pinref part="J87" gate="G$1" pin="GND@7"/>
 <wire x1="86.36" y1="190.5" x2="88.9" y2="190.5" width="0.1524" layer="91"/>
 <junction x="88.9" y="190.5"/>
-<pinref part="U1" gate="G$1" pin="GND@5"/>
+<pinref part="J87" gate="G$1" pin="GND@5"/>
 <wire x1="86.36" y1="208.28" x2="88.9" y2="208.28" width="0.1524" layer="91"/>
 <junction x="88.9" y="208.28"/>
-<pinref part="U1" gate="G$1" pin="GND@4"/>
+<pinref part="J87" gate="G$1" pin="GND@4"/>
 <wire x1="86.36" y1="215.9" x2="88.9" y2="215.9" width="0.1524" layer="91"/>
 <junction x="88.9" y="215.9"/>
-<pinref part="U1" gate="G$1" pin="GND@6"/>
+<pinref part="J87" gate="G$1" pin="GND@6"/>
 <wire x1="86.36" y1="195.58" x2="88.9" y2="195.58" width="0.1524" layer="91"/>
 <junction x="88.9" y="195.58"/>
@@
 <label x="91.44" y="193.04" size="1.27" layer="95" xref="yes"/>
 <wire x1="86.36" y1="193.04" x2="91.44" y2="193.04" width="0.1524" layer="91"/>
-<pinref part="U1" gate="G$1" pin="GPIO12"/>
+<pinref part="J87" gate="G$1" pin="GPIO12"/>
 </segment>
 </net>
@@
 <wire x1="86.36" y1="220.98" x2="91.44" y2="220.98" width="0.1524" layer="91"/>
 <label x="91.44" y="220.98" size="1.27" layer="95" xref="yes"/>
-<pinref part="U1" gate="G$1" pin="RXD0/GPIO15"/>
+<pinref part="J87" gate="G$1" pin="RXD0/GPIO15"/>
 </segment>
 </net>
@@
 <wire x1="86.36" y1="223.52" x2="91.44" y2="223.52" width="0.1524" layer="91"/>
 <label x="91.44" y="223.52" size="1.27" layer="95" xref="yes"/>
-<pinref part="U1" gate="G$1" pin="TXD0/GPIO14"/>
+<pinref part="J87" gate="G$1" pin="TXD0/GPIO14"/>
 </segment>
 </net>
@@
 <net name="!PWR_LOSS" class="0">
 <segment>
-<pinref part="U1" gate="G$1" pin="GPIO26"/>
+<pinref part="J87" gate="G$1" pin="GPIO26"/>
 <wire x1="38.1" y1="185.42" x2="33.02" y2="185.42" width="0.1524" layer="91"/>
 <label x="33.02" y="185.42" size="1.27" layer="95" rot="R180" xref="yes"/>
@@
 <wire x1="38.1" y1="218.44" x2="33.02" y2="218.44" width="0.1524" layer="91"/>
 <label x="33.02" y="218.44" size="1.27" layer="95" rot="R180" xref="yes"/>
-<pinref part="U1" gate="G$1" pin="GPIO17/GEN0"/>
+<pinref part="J87" gate="G$1" pin="GPIO17/GEN0"/>
 </segment>
 </net>
 <net name="3V3" class="0">
 <segment>
-<pinref part="U1" gate="G$1" pin="3V3@1"/>
+<pinref part="J87" gate="G$1" pin="3V3@1"/>
 <wire x1="38.1" y1="231.14" x2="20.32" y2="231.14" width="0.1524" layer="91"/>
 <wire x1="20.32" y1="231.14" x2="20.32" y2="233.68" width="0.1524" layer="91"/>
-<pinref part="U1" gate="G$1" pin="3V3@2"/>
+<pinref part="J87" gate="G$1" pin="3V3@2"/>
 <wire x1="38.1" y1="210.82" x2="20.32" y2="210.82" width="0.1524" layer="91"/>
 <wire x1="20.32" y1="210.82" x2="20.32" y2="231.14" width="0.1524" layer="91"/>
@@
 <wire x1="38.1" y1="223.52" x2="33.02" y2="223.52" width="0.1524" layer="91"/>
 <label x="33.02" y="223.52" size="1.27" layer="95" rot="R180" xref="yes"/>
-<pinref part="U1" gate="G$1" pin="GPIO4/GCKL"/>
+<pinref part="J87" gate="G$1" pin="GPIO4/GCKL"/>
 </segment>
 </net>
@@
 </segment>
 <segment>
-<pinref part="U1" gate="G$1" pin="5V0@2"/>
+<pinref part="J87" gate="G$1" pin="5V0@2"/>
 <wire x1="86.36" y1="228.6" x2="88.9" y2="228.6" width="0.1524" layer="91"/>
-<pinref part="U1" gate="G$1" pin="5V0@1"/>
+<pinref part="J87" gate="G$1" pin="5V0@1"/>
 <wire x1="86.36" y1="231.14" x2="88.9" y2="231.14" width="0.1524" layer="91"/>
 <wire x1="88.9" y1="231.14" x2="88.9" y2="233.68" width="0.1524" layer="91"/>
@@
 </segment>
 <segment>
-<pinref part="U1" gate="G$1" pin="GPIO27/GEN2"/>
+<pinref part="J87" gate="G$1" pin="GPIO27/GEN2"/>
 <wire x1="38.1" y1="215.9" x2="33.02" y2="215.9" width="0.1524" layer="91"/>
 <label x="33.02" y="215.9" size="1.27" layer="95" rot="R180" xref="yes"/>

Commit message: Added some stuff
Added clamps to RFID, added 1206 series resistor to LCD backlight
power in connector updated
lipo connector moved
played with cut away of plane
Parts:
- removed SJ4: JUMPER-PAD-2-NC_BY_TRACE, MakeItLabs:SOLDERJUMPER_CLOSED10MIL
- added D1, D4: BAT54S, MakeItLabs:BAT54S
- added R10: 100R, MakeItLabs:RESISTOR0603
- added R9: 10R, MakeItLabs:RESISTOR1206
- J100: value (none) -> PHOENIX1803426; device MakeItLabs:TERMBLOCK_1X2 -> MakeItLabs:PHOENIX1803426
Connections:
- removed net N$26: LCD3.LED+, LCD3.VCC, SJ4.1
- new net N$10: J5.4, R10.2
- new net N$9: LCD3.LED+, R9.2
- net +3.3V: now also LCD3.VCC, R9.1; no longer SJ4.2
- net +5VB: now also D1.C2, D4.C2
- net +5VIN: now also J100.2; no longer J100.1
- net GND: now also D1.A1, D4.A1, J100.1; no longer J100.2
- net RFID_RX: now also D4.C1A2, R10.1; no longer J5.4
- net RFID_TX: now also D1.C1A2
Other:
- moved on the sheet: C1, C25, J100

Commit message: moved stuff for Steve
Parts:
- removed J200: (no value), MakeItLabs:TERMBLOCK_1X2
- removed JP1: (no value), MakeItLabs:PINHD-2X8
- removed SJ3: JUMPER-PAD-2-NC_BY_TRACE, MakeItLabs:SOLDERJUMPER_CLOSED10MIL
- added J3: (no value), MakeItLabs:PINHD-2X8SHROUD
- added JP4: (no value), MakeItLabs:M02POLAR
Connections:
- removed net N$3: LCD3.GND, SJ3.1
- net +3.3V: now also D1.C2, D4.C2, J3.8; no longer JP1.8
- net +5VB: no longer D1.C2, D4.C2
- net +5VIN: now also J3.4; no longer JP1.4
- net GND: now also J3.2, J3.6, LCD3.GND; no longer JP1.2, JP1.6, SJ3.2
- net I2C_SCL: now also J3.15; no longer JP1.15
- net I2C_SDA: now also J3.13; no longer JP1.13
- net IN0P: now also J3.16; no longer JP1.16
- net IN1P: now also J3.14; no longer JP1.14
- net IN2P: now also J3.12; no longer JP1.12
- net IN3P: now also J3.10; no longer JP1.10
- net N$6: now also JP4.2; no longer J200.1
- net N$7: now also JP4.1; no longer J200.2
- net OUT0P: now also J3.1; no longer JP1.1
- net OUT1P: now also J3.3; no longer JP1.3
- net OUT2P: now also J3.5; no longer JP1.5
- net OUT3P: now also J3.7; no longer JP1.7
- net RFID_RX: now also J3.11; no longer JP1.11
- net RFID_TX: now also J3.9; no longer JP1.9
