File: hardware/doorbot/REV0/doorbot/doorbot.kicad_pcb (KiCad board)
At the start: 2 copper layers, 65 x 56.5 mm, 64 parts, among them J1 Raspberry_Pi_2_3, J2 Screw_Terminal_01x12, J3 PoE Passthrough, Q1 2N7002, U1 ATmega328P-AU, U10 TLP291, U2 TLP291, U3 TLP291, U4 TLP291, U5 TLP291, U6 TLP291, U7 DRV103, U8 MC78L05_SOT89, U9 TLP291, Y1 16MHz

Commit message: more doorbot pcb work
Parts:
- added C10: .1uF, Capacitors_SMD:C_0603, B.Cu at (108.6, 88.9)
- added C9: 1uF, Capacitors_SMD:CP_Elec_3x5.3, B.Cu at (111.8, 80.0)
- added D5: BAT54S, TO_SOT_Packages_SMD:SOT-23, B.Cu at (119.4, 80.0)
- added D6: BAT54S, TO_SOT_Packages_SMD:SOT-23, B.Cu at (108.6, 108.6)
- added D7: BAT54S, TO_SOT_Packages_SMD:SOT-23, B.Cu at (108.6, 103.5)
- added J4: Conn_01x03, Pin_Headers:Pin_Header_Straight_1x03_Pitch2.54mm, F.Cu at (109.2, 82.5)
- added J5: Conn_01x04, Pin_Headers:Pin_Header_Straight_1x04_Pitch2.54mm, F.Cu at (109.2, 91.4)
- C3, C4, C5, C6: footprint Capacitor_SMD:C_0603_1608Metric -> Capacitors_SMD:C_0603
- moved R28 6.35 mm to (118.7, 101.6)
- moved U10 6.35 mm to (119.4, 95.2)
- moved R10 3.97 mm to (123.2, 88.9)
- moved R27 3.81 mm to (111.8, 101.6)
- moved U9 3.81 mm to (112.4, 95.2)
- moved R23 3.53 mm to (120.7, 88.9)
- moved C8 1.80 mm to (141.0, 87.6)
- moved C7 1.72 mm to (135.9, 87.6), turned to 90 degrees
- moved Y1 1.54 mm to (138.4, 87.6)
Connections:
- U1 pad 23: Net-(U1-Pad23) -> RGB_DATA
Routing:
- net Net-(D6-Pad3): track 0.00 -> 56.6 mm, vias 0 -> 2
- net Net-(D7-Pad3): track 0.00 -> 46.4 mm, vias 0 -> 2
- net +3V3: track 62.1 -> 91.7 mm, vias 2 -> 4
- net RGB_DATA: track 0.00 -> 16.2 mm
- net +5V: track 53.5 -> 67.9 mm, vias 1 -> 2
- net Net-(R26-Pad1): track 101.4 -> 89.3 mm
- net /WG_LED_RAW: track 20.1 -> 13.8 mm
- net Earth: track 19.1 -> 24.9 mm
- net /WG_BEEP_RAW: track 20.8 -> 17.0 mm
- net Net-(R25-Pad1): track 100.8 -> 97.8 mm
- net Net-(R6-Pad1): track 47.7 -> 45.0 mm
- net Net-(R10-Pad2): track 7.79 -> 5.52 mm
- net DOOR_SW: track 54.9 -> 52.9 mm
- net WG_D0: track 30.6 -> 28.6 mm
- net GND: track 67.6 -> 65.6 mm, vias 8 -> 9
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
Commit message: doorbot pcb rev0 draft 2 ready for review
Parts:
- added C11: 1uF, Capacitors_SMD:CP_Elec_3x5.3, B.Cu at (109.2, 107.3)
- added C12: .1uF, Capacitors_SMD:C_0603, B.Cu at (107.3, 81.9)
- added D8: BAT54S, TO_SOT_Packages_SMD:SOT-23, B.Cu at (119.5, 80.2)
- added G***: LOGO, doorbot_pcb_library:makeit-logo, F.Cu at (139.1, 73.7)
- added R32: 4.7K, Resistors_SMD:R_0603, B.Cu at (107.3, 76.2)
- added R33: 4.7K, Resistors_SMD:R_0603, B.Cu at (115.6, 80.0)
- added RV1: 100K, Potentiometers:Potentiometer_Trimmer_Bourns_3269P, F.Cu at (165.7, 89.5)
- J4: value Conn_01x03 -> Conn_01x04; footprint Pin_Headers:Pin_Header_Straight_1x03_Pitch2.54mm -> Connect:Grove_1x04
- J5: footprint Pin_Headers:Pin_Header_Straight_1x04_Pitch2.54mm -> Connect:Grove_1x04
- moved D6 14.0 mm to (108.6, 94.6), turned to 90 degrees
- moved C10 13.4 mm to (107.3, 102.2), turned to 270 degrees
- moved D7 6.84 mm to (114.9, 101.0), turned to 90 degrees
- moved D5 5.99 mm to (114.3, 76.8), turned to 270 degrees
- moved J4 5.72 mm to (109.2, 76.8), turned to 0 degrees
- moved J5 5.72 mm to (109.2, 97.2)
- moved C9 2.84 mm to (113.0, 82.5), turned to 270 degrees
- moved LED2 1.27 mm to (109.9, 73.0)
- renumbered D3 to LED1, D2 to LED2, D4 to LED3
Connections:
- D5 pad 3: RGB_DATA -> AT_SCL
- D6 pad 3: Net-(D6-Pad3) -> PI_SCL
- D7 pad 3: Net-(D7-Pad3) -> PI_SDA
- J1 pad 3: Net-(D6-Pad3) -> PI_SDA
- J1 pad 5: Net-(D7-Pad3) -> PI_SCL
- J4 pad 1: +5V -> AT_SCL
- J4 pad 2: RGB_DATA -> AT_SDA
- J4 pad 3: GND -> +5V
- J5 pad 1: +3V3 -> PI_SCL
- J5 pad 2: Net-(D6-Pad3) -> PI_SDA
- J5 pad 3: Net-(D7-Pad3) -> +3V3
- U1 pad 23: RGB_DATA -> Net-(U1-Pad23)
- U1 pad 27: Net-(U1-Pad27) -> AT_SDA
- U1 pad 28: Net-(U1-Pad28) -> AT_SCL
Routing:
- net Net-(D6-Pad3): track 56.6 -> 0.00 mm, vias 2 -> 0
- net Net-(D7-Pad3): track 46.4 -> 0.00 mm, vias 2 -> 0
- net PI_SDA: track 0.00 -> 45.5 mm, vias 0 -> 1
- net PI_SCL: track 0.00 -> 42.5 mm, vias 0 -> 1
- net Earth: track 24.9 -> 49.8 mm, vias 7 -> 22
- net AT_SCL: track 0.00 -> 24.4 mm
- net AT_SDA: track 0.00 -> 20.9 mm
- net RGB_DATA: track 16.2 -> 0.00 mm
- net GND: track 65.6 -> 78.6 mm, vias 9 -> 50
- net Net-(R13-Pad1): track 11.1 -> 23.0 mm, vias 0 -> 1
- net +3V3: track 91.7 -> 102.0 mm, vias 4 -> 6
- net +5V: track 67.9 -> 75.6 mm, vias 2 -> 3
- net Net-(R25-Pad1): track 97.8 -> 102.6 mm
- net Net-(J1-Pad33): track 58.4 -> 61.1 mm
Other:
- board text added: "+12V"
- board text added: "12V"
- board text added: "A"
- board text added: "ALRM.SW"
- board text added: "ATMEGA GROVE"
- board text added: "B"
- board text added: "BEEP"
- board text added: "D0"
- board text added: "D1"
- board text added: "DOORBOT - RFID ALL THE THINGS"
- board text added: "DUTY CYCLE"
- board text added: "GND"
- board text added: "LED"
- board text added: "PI GROVE"
- board text added: "PWR IN"
- board text added: "REV0 2019.03.22 - STEVE RICHARDSON"
- board text added: "SOLENOID"
- board text added: "WIEGAND RFID"
- board text removed: "PWR.12V"
- board text removed: "PWR.GND"
- board text removed: "R.12V"
- board text removed: "R.D0"
- board text removed: "R.D1"
- board text removed: "R.GND"
- board text removed: "SOL.A"
- board text removed: "SOL.B"
- board text removed: "SW.A"
- board text removed: "SW.B"
