File: hardware/doorbot/REV0/doorbot/doorbot.sch (KiCad schematic (older format))
At the start: 36 parts, among them J1 Raspberry_Pi_2_3, J2 Screw_Terminal_01x12, J3 Conn_02x02_Odd_Even, Q1 2N7002, U1 ATmega328P-AU, U2 TLP291, U3 TLP291, U4 TLP291, U5 TLP291, U6 TLP291, U7 DRV103, U8 L78L05_SO8

Commit message: more doorbot schematic & pcb work
Parts:
- removed U8: L78L05_SO8, Package_SO:SOIC-8_3.9x4.9mm_P1.27mm, symbol Regulator_Linear:L78L05_SO8
- added R19, R20, R21, R22: 47, Resistors_SMD:R_0603, symbol Device:R_Small_US
- added U8: MC78L05_SOT89, TO_SOT_Packages_SMD:SOT-89-3_Handsoldering, symbol Regulator_Linear:MC78L05_SOT89
- C2: footprint (none) -> Capacitors_SMD:CP_Elec_3x5.3
- J3: value Conn_02x02_Odd_Even -> PoE Passthrough
- R1, R10, R11, R12, R13, R14, R15, R16, R18, R2, R3, R5, R6, R7, R8, R9: footprint Resistor_SMD:R_0603_1608Metric -> Resistors_SMD:R_0603
- R17: value R_Small_US -> 100; footprint Resistor_SMD:R_0603_1608Metric -> Resistors_SMD:R_0603
- R4: value 10 -> 47; footprint Resistor_SMD:R_0603_1608Metric -> Resistors_SMD:R_0603
- U7: symbol doorbot:DRV103 -> doorbot-rescue:DRV103-doorbot
Connections:
- net labels added: AT_MISO, AT_MOSI, AT_RST, AT_SCK, ICSP_MISO, ICSP_MOSI, ICSP_RESET, ICSP_SCK, WG_D0_RAW, WG_D1_RAW
- wire segments 129 -> 143
Other:
- note added: "https://learn.adafruit.com/program-an-avr-or-arduino-using-raspberry-pi-gpio-pins/overview"
Changed lines of the file:
@@
 EESchema Schematic File Version 4
 LIBS:doorbot-cache
-EELAYER 26 0
+EELAYER 29 0
 EELAYER END
 $Descr A4 11693 8268
@@
 Text Label 2900 6300 0    50   ~ 0
 AT_RXD
-$Comp
-L Device:R_Small_US R1
-U 1 1 5C8E9583
-P 3700 6200
-F 0 "R1" V 3600 6200 50  0000 C CNN
-F 1 "1K" V 3800 6200 50  0000 C CNN
-F 2 "Resistor_SMD:R_0603_1608Metric" H 3700 6200 50  0001 C CNN
-F 3 "~" H 3700 6200 50  0001 C CNN
-	1    3700 6200
-	0    1    1    0
-$EndComp
-$Comp
-L Device:R_Small_US R2
-U 1 1 5C8E962E
-P 3850 6400
-F 0 "R2" V 3750 6400 50  0000 C CNN
-F 1 "1K" V 3950 6400 50  0000 C CNN
-F 2 "Resistor_SMD:R_0603_1608Metric" H 3850 6400 50  0001 C CNN
-F 3 "~" H 3850 6400 50  0001 C CNN
-	1    3850 6400
-	0    1    1    0
-$EndComp
 Wire Wire Line
 	3350 6300 3350 6200
@@
 F 0 "R11" H 6868 4796 50  0000 L CNN
 F 1 "4.7K" H 6868 4705 50  0000 L CNN
-F 2 "Resistor_SMD:R_0603_1608Metric" H 6800 4750 50  0001 C CNN
+F 2 "Resistors_SMD:R_0603" H 6800 4750 50  0001 C CNN
 F 3 "~" H 6800 4750 50  0001 C CNN
 	1    6800 4750
@@
 F 0 "R12" H 6868 5346 50  0000 L CNN
 F 1 "4.7K" H 6868 5255 50  0000 L CNN
-F 2 "Resistor_SMD:R_0603_1608Metric" H 6800 5300 50  0001 C CNN
+F 2 "Resistors_SMD:R_0603" H 6800 5300 50  0001 C CNN
 F 3 "~" H 6800 5300 50  0001 C CNN
 	1    6800 5300
@@
 Connection ~ 2200 4200
 $Comp
-L doorbot:DRV103 U7
+L doorbot-rescue:DRV103-doorbot U7
 U 1 1 5C8F15EA
 P 7900 1500
@@
 Wire Wire Line
 	8700 2300 8700 2200
-$Comp
-L Regulator_Linear:L78L05_SO8 U8
-U 1 1 5C8F790B
-P 9350 950
-F 0 "U8" H 9350 1192 50  0000 C CNN
-F 1 "L78L05_SO8" H 9350 1101 50  0000 C CNN
-F 2 "Package_SO:SOIC-8_3.9x4.9mm_P1.27mm" H 9450 1150 50  0001 C CIN
-F 3 "http://www.st.com/content/ccc/resource/technical/document/datasheet/15/55/e5/aa/23/5b/43/fd/CD00000446.pdf/files/CD00000446.pdf/jcr:content/translations/en.CD00000446.pdf" H 9550 950 50  0001 C CNN
-	1    9350 950
-	1    0    0    -1
-$EndComp
 Wire Wire Line
 	8700 1400 8700 1000
@@
 F 0 "R8" V 6445 2550 50  0000 C CNN
 F 1 "1K" V 6536 2550 50  0000 C CNN
-F 2 "Resistor_SMD:R_0603_1608Metric" H 6650 2550 50  0001 C CNN
+F 2 "Resistors_SMD:R_0603" H 6650 2550 50  0001 C CNN
 F 3 "~" H 6650 2550 50  0001 C CNN
 	1    6650 2550
@@
 F 0 "R7" H 6568 2196 50  0000 L CNN
 F 1 "4.7K" H 6568 2105 50  0000 L CNN
-F 2 "Resistor_SMD:R_0603_1608Metric" H 6500 2150 50  0001 C CNN
+F 2 "Resistors_SMD:R_0603" H 6500 2150 50  0001 C CNN
 F 3 "~" H 6500 2150 50  0001 C CNN
 	1    6500 2150
@@
 F 0 "R15" H 7218 2196 50  0000 L CNN
 F 1 "4.7K" H 7218 2105 50  0000 L CNN
-F 2 "Resistor_SMD:R_0603_1608Metric" H 7150 2150 50  0001 C CNN
+F 2 "Resistors_SMD:R_0603" H 7150 2150 50  0001 C CNN
 F 3 "~" H 7150 2150 50  0001 C CNN
 	1    7150 2150
@@
 F 0 "R13" V 6895 1000 50  0000 C CNN
 F 1 "R_PWM" V 6986 1000 50  0000 C CNN
-F 2 "Resistor_SMD:R_0603_1608Metric" H 7100 1000 50  0001 C CNN
+F 2 "Resistors_SMD:R_0603" H 7100 1000 50  0001 C CNN
 F 3 "~" H 7100 1000 50  0001 C CNN
 	1    7100 1000
@@
 F 0 "R14" V 6895 1800 50  0000 C CNN
 F 1 "R_FREQ" V 6986 1800 50  0000 C CNN
-F 2 "Resistor_SMD:R_0603_1608Metric" H 7100 1800 50  0001 C CNN
+F 2 "Resistors_SMD:R_0603" H 7100 1800 50  0001 C CNN
 F 3 "~" H 7100 1800 50  0001 C CNN
 	1    7100 1800
@@
 F 0 "C2" H 8415 1246 50  0000 L CNN
 F 1 "1uF" H 8415 1155 50  0000 L CNN
-F 2 "" H 8300 1200 50  0001 C CNN
+F 2 "Capacitors_SMD:CP_Elec_3x5.3" H 8300 1200 50  0001 C CNN
 F 3 "~" H 8300 1200 50  0001 C CNN
 	1    8300 1200
@@
 F 0 "R9" H 6868 3146 50  0000 L CNN
 F 1 "R_LED" H 6868 3055 50  0000 L CNN
-F 2 "Resistor_SMD:R_0603_1608Metric" H 6800 3100 50  0001 C CNN
+F 2 "Resistors_SMD:R_0603" H 6800 3100 50  0001 C CNN
 F 3 "~" H 6800 3100 50  0001 C CNN
 	1    6800 3100
@@
 F 0 "R6" V 5295 2550 50  0000 C CNN
 F 1 "47" V 5386 2550 50  0000 C CNN
-F 2 "Resistor_SMD:R_0603_1608Metric" H 5500 2550 50  0001 C CNN
+F 2 "Resistors_SMD:R_0603" H 5500 2550 50  0001 C CNN
 F 3 "~" H 5500 2550 50  0001 C CNN
 	1    5500 2550
@@
 F 0 "R5" H 5468 3146 50  0000 L CNN
 F 1 "4.7K" H 5468 3055 50  0000 L CNN
-F 2 "Resistor_SMD:R_0603_1608Metric" H 5400 3100 50  0001 C CNN
+F 2 "Resistors_SMD:R_0603" H 5400 3100 50  0001 C CNN
 F 3 "~" H 5400 3100 50  0001 C CNN
 	1    5400 3100
@@
 Wire Wire Line
 	5850 2550 5600 2550
-Wire Wire Line
-	2900 3000 5050 3000
-Wire Wire Line
-	5050 3000 5050 2550
 Wire Wire Line
 	5050 2550 5400 2550
@@
 F 0 "R18" H 8282 4004 50  0000 R CNN
 F 1 "470" H 8282 4095 50  0000 R CNN
-F 2 "Resistor_SMD:R_0603_1608Metric" H 8350 4050 50  0001 C CNN
+F 2 "Resistors_SMD:R_0603" H 8350 4050 50  0001 C CNN
 F 3 "~" H 8350 4050 50  0001 C CNN
 	1    8350 4050
@@
 P 4800 3250
 F 0 "R4" V 4700 3250 50  0000 C CNN
-F 1 "10" V 4900 3250 50  0000 C CNN
-F 2 "Resistor_SMD:R_0603_1608Metric" H 4800 3250 50  0001 C CNN
+F 1 "47" V 4900 3250 50  0000 C CNN
+F 2 "Resistors_SMD:R_0603" H 4800 3250 50  0001 C CNN
 F 3 "~" H 4800 3250 50  0001 C CNN
 	1    4800 3250
 	0    1    1    0
 $EndComp
-Wire Wire Line
-	4700 3250 3150 3250
-Wire Wire Line
-	3150 3250 3150 3100
-Wire Wire Line
-	3150 3100 2900 3100
 $Comp
 L power:+3.3V #PWR07
@@
 F 0 "R16" V 8050 4850 50  0000 C CNN
 F 1 "100" V 8250 4850 50  0000 C CNN
-F 2 "Resistor_SMD:R_0603_1608Metric" H 8150 4850 50  0001 C CNN
+F 2 "Resistors_SMD:R_0603" H 8150 4850 50  0001 C CNN
 F 3 "~" H 8150 4850 50  0001 C CNN
 	1    8150 4850
@@
 P 8150 5400
 F 0 "R17" V 8050 5400 50  0000 C CNN
-F 1 "R_Small_US" V 8250 5400 50  0000 C CNN
-F 2 "Resistor_SMD:R_0603_1608Metric" H 8150 5400 50  0001 C CNN
+F 1 "100" V 8250 5400 50  0000 C CNN
+F 2 "Resistors_SMD:R_0603" H 8150 5400 50  0001 C CNN
 F 3 "~" H 8150 5400 50  0001 C CNN
 	1    8150 5400
@@
 F 0 "R10" H 6868 4196 50  0000 L CNN
 F 1 "4.7K" H 6868 4105 50  0000 L CNN
-F 2 "Resistor_SMD:R_0603_1608Metric" H 6800 4150 50  0001 C CNN
+F 2 "Resistors_SMD:R_0603" H 6800 4150 50  0001 C CNN
 F 3 "~" H 6800 4150 50  0001 C CNN
 	1    6800 4150
@@
 F 0 "R3" H 4018 6646 50  0000 L CNN
 F 1 "2K" H 4018 6555 50  0000 L CNN
-F 2 "Resistor_SMD:R_0603_1608Metric" H 3950 6600 50  0001 C CNN
+F 2 "Resistors_SMD:R_0603" H 3950 6600 50  0001 C CNN
 F 3 "~" H 3950 6600 50  0001 C CNN
 	1    3950 6600
@@
 P 3450 850
 F 0 "J3" H 3500 1067 50  0000 C CNN
-F 1 "Conn_02x02_Odd_Even" H 3500 976 50  0000 C CNN
+F 1 "PoE Passthrough" H 3500 976 50  0000 C CNN
 F 2 "Connector_PinHeader_2.54mm:PinHeader_2x02_P2.54mm_Vertical" H 3450 850 50  0001 C CNN
 F 3 "~" H 3450 850 50  0001 C CNN
@@
 	1    0    0    -1
 $EndComp
+$Comp
+L Regulator_Linear:MC78L05_SOT89 U8
+U 1 1 5C8FEE6D
+P 9350 950
+F 0 "U8" H 9350 1192 50  0000 C CNN
+F 1 "MC78L05_SOT89" H 9350 1101 50  0000 C CNN
+F 2 "TO_SOT_Packages_SMD:SOT-89-3_Handsoldering" H 9350 1150 50  0001 C CIN
+F 3 "http://www.fairchildsemi.com/ds/LM/LM78L05A.pdf" H 9350 900 50  0001 C CNN
+	1    9350 950
+	1    0    0    -1
+$EndComp
+Text Label 9250 4850 0    50   ~ 0
+WG_D0_RAW
+Text Label 9250 4950 0    50   ~ 0
+WG_D1_RAW
+Wire Wire Line
+	2900 1700 5050 1700
+Wire Wire Line
+	5050 1700 5050 2550
+Wire Wire Line
+	4700 3250 4600 3250
+Wire Wire Line
+	4600 3250 4600 1800
+Wire Wire Line
+	4600 1800 2900 1800
+Wire Wire Line
+	2800 4900 3300 4900
+Wire Wire Line
+	2800 5000 3550 5000
+Wire Wire Line
+	2800 5100 3800 5100
+$Comp
+L Device:R_Small_US R19
+U 1 1 5CA21261
+P 3400 4900
+F 0 "R19" V 3195 4900 50  0000 C CNN
+F 1 "47" V 3286 4900 50  0000 C CNN
+F 2 "Resistors_SMD:R_0603" H 3400 4900 50  0001 C CNN
+F 3 "~" H 3400 4900 50  0001 C CNN
+	1    3400 4900
+	0    1    1    0
+$EndComp
+$Comp
+L Device:R_Small_US R20
+U 1 1 5CA224AA
+P 3650 5000
+F 0 "R20" V 3400 5000 50  0000 C CNN
+F 1 "47" V 3500 5000 50  0000 C CNN
+F 2 "Resistors_SMD:R_0603" H 3650 5000 50  0001 C CNN
+F 3 "~" H 3650 5000 50  0001 C CNN
+	1    3650 5000
+	0    1    1    0
+$EndComp
+$Comp
+L Device:R_Small_US R21
+U 1 1 5CA22D34
+P 3900 5100
+F 0 "R21" V 4000 5100 50  0000 C CNN
+F 1 "47" V 4100 5100 50  0000 C CNN
+F 2 "Resistors_SMD:R_0603" H 3900 5100 50  0001 C CNN
+F 3 "~" H 3900 5100 50  0001 C CNN
+	1    3900 5100
+	0    1    1    0
+$EndComp
+Wire Wire Line
+	3500 4900 4450 4900
+Wire Wire Line
+	3750 5000 4450 5000
+Wire Wire Line
+	4000 5100 4450 5100
+Text Label 4050 4900 0    50   ~ 0
+ICSP_MOSI
+Text Label 4050 5000 0    50   ~ 0
+ICSP_MISO
+Text Label 4050 5100 0    50   ~ 0
+ICSP_SCK
+$Comp
+L Device:R_Small_US R22
+U 1 1 5CA55E32
+P 3900 5800
+F 0 "R22" V 4000 5800 50  0000 C CNN
+F 1 "47" V 4100 5800 50  0000 C CNN
+F 2 "Resistors_SMD:R_0603" H 3900 5800 50  0001 C CNN
+F 3 "~" H 3900 5800 50  0001 C CNN
+	1    3900 5800
+	0    1    1    0
+$EndComp
+Wire Wire Line
+	4000 5800 4450 5800
+Text Label 4050 5800 0    50   ~ 0
+ICSP_RESET
+Wire Wire Line
+	3800 5800 3350 5800
+Wire Wire Line
+	3350 5800 3350 6100
+Wire Wire Line
+	3350 6100 2800 6100
+Text Label 2950 4900 0    50   ~ 0
+AT_MOSI
+Text Label 2950 5000 0    50   ~ 0
+AT_MISO
+Text Label 2950 5100 0    50   ~ 0
+AT_SCK
+Text Label 2900 6100 0    50   ~ 0
+AT_RST
+Wire Wire Line
+	2900 3000 3750 3000
+Wire Wire Line
+	1300 2700 750  2700
+Wire Wire Line
+	1300 2600 750  2600
+Wire Wire Line
+	1300 1900 750  1900
+Text Label 3250 3000 0    50   ~ 0
+ICSP_RESET
+Text Label 800  2700 0    50   ~ 0
+ICSP_SCK
+Text Label 800  2600 0    50   ~ 0
+ICSP_MOSI
+Text Label 800  1900 0    50   ~ 0
+ICSP_MISO
+$Comp
+L Device:R_Small_US R2
+U 1 1 5C8E962E
+P 3850 6400
+F 0 "R2" V 3750 6400 50  0000 C CNN
+F 1 "1K" V 3950 6400 50  0000 C CNN
+F 2 "Resistors_SMD:R_0603" H 3850 6400 50  0001 C CNN
+F 3 "~" H 3850 6400 50  0001 C CNN
+	1    3850 6400
+	0    1    1    0
+$EndComp
+$Comp
+L Device:R_Small_US R1
+U 1 1 5C8E9583
+P 3700 6200
+F 0 "R1" V 3600 6200 50  0000 C CNN
+F 1 "1K" V 3800 6200 50  0000 C CNN
+F 2 "Resistors_SMD:R_0603" H 3700 6200 50  0001 C CNN
+F 3 "~" H 3700 6200 50  0001 C CNN
+	1    3700 6200
+	0    1    1    0
+$EndComp
+Text Notes 1150 7650 0    50   ~ 0
+https://learn.adafruit.com/program-an-avr-or-arduino-using-raspberry-pi-gpio-pins/overview
 $EndSCHEMATC

Commit message: moar doorbot pcb
Parts:
- added R23: 47, Resistor_SMD:R_0603_1608Metric, symbol Device:R_Small_US
- R1, R10, R11, R12, R13, R14, R15, R16, R17, R18, R19, R2, R20, R21, R22, R3, R4, R5, R6, R7, R8, R9: footprint Resistors_SMD:R_0603 -> Resistor_SMD:R_0603_1608Metric
Connections:
- wire segments 143 -> 146
Changed lines of the file:
@@
 F 0 "R11" H 6868 4796 50  0000 L CNN
 F 1 "4.7K" H 6868 4705 50  0000 L CNN
-F 2 "Resistors_SMD:R_0603" H 6800 4750 50  0001 C CNN
+F 2 "Resistor_SMD:R_0603_1608Metric" H 6800 4750 50  0001 C CNN
 F 3 "~" H 6800 4750 50  0001 C CNN
 	1    6800 4750
@@
 F 0 "R12" H 6868 5346 50  0000 L CNN
 F 1 "4.7K" H 6868 5255 50  0000 L CNN
-F 2 "Resistors_SMD:R_0603" H 6800 5300 50  0001 C CNN
+F 2 "Resistor_SMD:R_0603_1608Metric" H 6800 5300 50  0001 C CNN
 F 3 "~" H 6800 5300 50  0001 C CNN
 	1    6800 5300
@@
 F 0 "R8" V 6445 2550 50  0000 C CNN
 F 1 "1K" V 6536 2550 50  0000 C CNN
-F 2 "Resistors_SMD:R_0603" H 6650 2550 50  0001 C CNN
+F 2 "Resistor_SMD:R_0603_1608Metric" H 6650 2550 50  0001 C CNN
 F 3 "~" H 6650 2550 50  0001 C CNN
 	1    6650 2550
@@
 F 0 "R7" H 6568 2196 50  0000 L CNN
 F 1 "4.7K" H 6568 2105 50  0000 L CNN
-F 2 "Resistors_SMD:R_0603" H 6500 2150 50  0001 C CNN
+F 2 "Resistor_SMD:R_0603_1608Metric" H 6500 2150 50  0001 C CNN
 F 3 "~" H 6500 2150 50  0001 C CNN
 	1    6500 2150
@@
 F 0 "R15" H 7218 2196 50  0000 L CNN
 F 1 "4.7K" H 7218 2105 50  0000 L CNN
-F 2 "Resistors_SMD:R_0603" H 7150 2150 50  0001 C CNN
+F 2 "Resistor_SMD:R_0603_1608Metric" H 7150 2150 50  0001 C CNN
 F 3 "~" H 7150 2150 50  0001 C CNN
 	1    7150 2150
@@
 F 0 "R13" V 6895 1000 50  0000 C CNN
 F 1 "R_PWM" V 6986 1000 50  0000 C CNN
-F 2 "Resistors_SMD:R_0603" H 7100 1000 50  0001 C CNN
+F 2 "Resistor_SMD:R_0603_1608Metric" H 7100 1000 50  0001 C CNN
 F 3 "~" H 7100 1000 50  0001 C CNN
 	1    7100 1000
@@
 F 0 "R14" V 6895 1800 50  0000 C CNN
 F 1 "R_FREQ" V 6986 1800 50  0000 C CNN
-F 2 "Resistors_SMD:R_0603" H 7100 1800 50  0001 C CNN
+F 2 "Resistor_SMD:R_0603_1608Metric" H 7100 1800 50  0001 C CNN
 F 3 "~" H 7100 1800 50  0001 C CNN
 	1    7100 1800
@@
 F 0 "R9" H 6868 3146 50  0000 L CNN
 F 1 "R_LED" H 6868 3055 50  0000 L CNN
-F 2 "Resistors_SMD:R_0603" H 6800 3100 50  0001 C CNN
+F 2 "Resistor_SMD:R_0603_1608Metric" H 6800 3100 50  0001 C CNN
 F 3 "~" H 6800 3100 50  0001 C CNN
 	1    6800 3100
@@
 F 0 "R6" V 5295 2550 50  0000 C CNN
 F 1 "47" V 5386 2550 50  0000 C CNN
-F 2 "Resistors_SMD:R_0603" H 5500 2550 50  0001 C CNN
+F 2 "Resistor_SMD:R_0603_1608Metric" H 5500 2550 50  0001 C CNN
 F 3 "~" H 5500 2550 50  0001 C CNN
 	1    5500 2550
@@
 F 0 "R5" H 5468 3146 50  0000 L CNN
 F 1 "4.7K" H 5468 3055 50  0000 L CNN
-F 2 "Resistors_SMD:R_0603" H 5400 3100 50  0001 C CNN
+F 2 "Resistor_SMD:R_0603_1608Metric" H 5400 3100 50  0001 C CNN
 F 3 "~" H 5400 3100 50  0001 C CNN
 	1    5400 3100
@@
 F 0 "R18" H 8282 4004 50  0000 R CNN
 F 1 "470" H 8282 4095 50  0000 R CNN
-F 2 "Resistors_SMD:R_0603" H 8350 4050 50  0001 C CNN
+F 2 "Resistor_SMD:R_0603_1608Metric" H 8350 4050 50  0001 C CNN
 F 3 "~" H 8350 4050 50  0001 C CNN
 	1    8350 4050
@@
 F 0 "R4" V 4700 3250 50  0000 C CNN
 F 1 "47" V 4900 3250 50  0000 C CNN
-F 2 "Resistors_SMD:R_0603" H 4800 3250 50  0001 C CNN
+F 2 "Resistor_SMD:R_0603_1608Metric" H 4800 3250 50  0001 C CNN
 F 3 "~" H 4800 3250 50  0001 C CNN
 	1    4800 3250
@@
 F 0 "R16" V 8050 4850 50  0000 C CNN
 F 1 "100" V 8250 4850 50  0000 C CNN
-F 2 "Resistors_SMD:R_0603" H 8150 4850 50  0001 C CNN
+F 2 "Resistor_SMD:R_0603_1608Metric" H 8150 4850 50  0001 C CNN
 F 3 "~" H 8150 4850 50  0001 C CNN
 	1    8150 4850
@@
 F 0 "R17" V 8050 5400 50  0000 C CNN
 F 1 "100" V 8250 5400 50  0000 C CNN
-F 2 "Resistors_SMD:R_0603" H 8150 5400 50  0001 C CNN
+F 2 "Resistor_SMD:R_0603_1608Metric" H 8150 5400 50  0001 C CNN
 F 3 "~" H 8150 5400 50  0001 C CNN
 	1    8150 5400
@@
 F 0 "R10" H 6868 4196 50  0000 L CNN
 F 1 "4.7K" H 6868 4105 50  0000 L CNN
-F 2 "Resistors_SMD:R_0603" H 6800 4150 50  0001 C CNN
+F 2 "Resistor_SMD:R_0603_1608Metric" H 6800 4150 50  0001 C CNN
 F 3 "~" H 6800 4150 50  0001 C CNN
 	1    6800 4150
@@
 F 0 "R3" H 4018 6646 50  0000 L CNN
 F 1 "2K" H 4018 6555 50  0000 L CNN
-F 2 "Resistors_SMD:R_0603" H 3950 6600 50  0001 C CNN
+F 2 "Resistor_SMD:R_0603_1608Metric" H 3950 6600 50  0001 C CNN
 F 3 "~" H 3950 6600 50  0001 C CNN
 	1    3950 6600
@@
 WG_D1_RAW
 Wire Wire Line
-	2900 1700 5050 1700
-Wire Wire Line
-	5050 1700 5050 2550
+	5050 2000 5050 2550
 Wire Wire Line
 	4700 3250 4600 3250
 Wire Wire Line
-	4600 3250 4600 1800
-Wire Wire Line
-	4600 1800 2900 1800
+	4600 3250 4600 2100
 Wire Wire Line
 	2800 4900 3300 4900
@@
 F 0 "R19" V 3195 4900 50  0000 C CNN
 F 1 "47" V 3286 4900 50  0000 C CNN
-F 2 "Resistors_SMD:R_0603" H 3400 4900 50  0001 C CNN
+F 2 "Resistor_SMD:R_0603_1608Metric" H 3400 4900 50  0001 C CNN
 F 3 "~" H 3400 4900 50  0001 C CNN
 	1    3400 4900
@@
 F 0 "R20" V 3400 5000 50  0000 C CNN
 F 1 "47" V 3500 5000 50  0000 C CNN
-F 2 "Resistors_SMD:R_0603" H 3650 5000 50  0001 C CNN
+F 2 "Resistor_SMD:R_0603_1608Metric" H 3650 5000 50  0001 C CNN
 F 3 "~" H 3650 5000 50  0001 C CNN
 	1    3650 5000
@@
 F 0 "R21" V 4000 5100 50  0000 C CNN
 F 1 "47" V 4100 5100 50  0000 C CNN
-F 2 "Resistors_SMD:R_0603" H 3900 5100 50  0001 C CNN
+F 2 "Resistor_SMD:R_0603_1608Metric" H 3900 5100 50  0001 C CNN
 F 3 "~" H 3900 5100 50  0001 C CNN
 	1    3900 5100
@@
 F 0 "R22" V 4000 5800 50  0000 C CNN
 F 1 "47" V 4100 5800 50  0000 C CNN
-F 2 "Resistors_SMD:R_0603" H 3900 5800 50  0001 C CNN
+F 2 "Resistor_SMD:R_0603_1608Metric" H 3900 5800 50  0001 C CNN
 F 3 "~" H 3900 5800 50  0001 C CNN
 	1    3900 5800
@@
 F 0 "R2" V 3750 6400 50  0000 C CNN
 F 1 "1K" V 3950 6400 50  0000 C CNN
-F 2 "Resistors_SMD:R_0603" H 3850 6400 50  0001 C CNN
+F 2 "Resistor_SMD:R_0603_1608Metric" H 3850 6400 50  0001 C CNN
 F 3 "~" H 3850 6400 50  0001 C CNN
 	1    3850 6400
@@
 F 0 "R1" V 3600 6200 50  0000 C CNN
 F 1 "1K" V 3800 6200 50  0000 C CNN
-F 2 "Resistors_SMD:R_0603" H 3700 6200 50  0001 C CNN
+F 2 "Resistor_SMD:R_0603_1608Metric" H 3700 6200 50  0001 C CNN
 F 3 "~" H 3700 6200 50  0001 C CNN
 	1    3700 6200
@@
 Text Notes 1150 7650 0    50   ~ 0
 https://learn.adafruit.com/program-an-avr-or-arduino-using-raspberry-pi-gpio-pins/overview
+Wire Wire Line
+	4600 2100 2900 2100
+Wire Wire Line
+	2900 2000 5050 2000
+$Comp
+L Device:R_Small_US R23
+U 1 1 5C929A86
+P 5350 4250
+F 0 "R23" V 5145 4250 50  0000 C CNN
+F 1 "47" V 5236 4250 50  0000 C CNN
+F 2 "Resistor_SMD:R_0603_1608Metric" H 5350 4250 50  0001 C CNN
+F 3 "~" H 5350 4250 50  0001 C CNN
+	1    5350 4250
+	0    1    1    0
+$EndComp
+Wire Wire Line
+	5250 4250 4450 4250
+Wire Wire Line
+	4450 4250 4450 2200
+Wire Wire Line
+	4450 2200 2900 2200
 $EndSCHEMATC
