File: hardware/doorbot/REV0/doorbot/doorbot.sch (KiCad schematic (older format))
At the start: 79 parts, among them J1 Raspberry_Pi_2_3, J2 Screw_Terminal_01x12, J3 PoE Passthrough, J4 Conn_01x04, J5 Conn_01x04, Q1 2N7002, U1 ATmega328P-AU, U10 TLP291, U2 TLP291, U3 TLP291, U4 TLP291, U5 TLP291, U6 TLP291, U7 DRV103, U8 MC78L05_SOT89, U9 TLP291, Y1 16MHz

Commit message: update placeholder resistors with calculated values
Parts:
- C1: value C_DELAY -> 1uF
- C7, C8: value 12pF -> 20pF
- D1: value B260 -> SS34-E3/57T
- R1: value 1K -> 47
- R13: value R_PWM -> DNP
- R14: value R_FREQ -> 47.5K
- R16, R17: value 100 -> 330
- R25, R26: value 100 -> 270
- R30: value 100 -> 220
- R6: value 47 -> 270
- R9: value R_LED -> 330
Other:
- note added: "DNP R13 WHEN USING RV1"
- note added: "DNP R24 IF USING BOOST CONVERTER"
