File: hardware/uratt/uratt/uratt.kicad_pcb (KiCad board)
At the start: 4 copper layers, 62 x 97.4 mm, 154 parts, among them J1 USB_B_Micro, J2 Micro_SD_Card, J3 Conn_01x10, J4 Conn_01x04, J5 Conn_01x04, J6 Conn_01x02, J7 Conn_01x02, J8 Conn_01x02, J9 Conn_01x10, Q1 MMBT3904, Q2 MMBT3904, Q3 DMP31D0U, Q4 2N7002, SW1 SW_Push, SW2 SW_Push, SW3 SW_Push, SW4 SW_SPDT, U1 SN65220, U2 CP2102N-A01-GQFN24, U3 ESP32-WROOM-32, U4 MCP73832-2-OT, U5 TPS2115A, U6 TPS61032PWP, U7 AP2112K-3.3, U8 AP2112K-3.3, U9 MP6513

Commit message: add rev0 fabrication files - pcb sent off to fab
Parts:
- added FB3: FB (OPTION), Inductor_SMD:L_0603_1608Metric, F.Cu at (80.5, 44.2)
- added FB4: FB, Inductor_SMD:L_0603_1608Metric, F.Cu at (84.1, 44.2)
- added JP5: 0 (OPTION), Resistor_SMD:R_0603_1608Metric, F.Cu at (35.3, 72.9)
- added JP6: 0 (OPTION), Resistor_SMD:R_0603_1608Metric, F.Cu at (38.1, 72.9)
- added R54: 4.7K, Resistor_SMD:R_0603_1608Metric, F.Cu at (70.6, 47.5)
- added R55: 4.7K, Resistor_SMD:R_0603_1608Metric, F.Cu at (76.7, 34.0)
- added TP7: TestPoint, TestPoint:TestPoint_Pad_D1.0mm, B.Cu at (38.4, 74.4)
- FB1, FB2: value FB -> FB (OPTION)
- J5: footprint Connector_JST:JST_PH_B4B-PH-K_1x04_P2.00mm_Vertical -> Connector:NS-Tech_Grove_1x04_P2mm_Vertical
- R17, R18: value 5K -> 4.7K
- SW3: footprint Button_Switch_SMD:SW_Push_1P1T_NO_CK_KMR2 -> Button_Switch_SMD:SW_Push_1P1T_NO_CK_KSC6xxJ
- moved Q4 16.3 mm to (71.1, 115.1)
- moved R52 13.3 mm to (70.9, 112.0), turned to 0 degrees
- moved J9 8.50 mm to (63.2, 102.3), turned to 270 degrees
- moved SW3 4.32 mm to (77.5, 112.3)
- moved J8 1.60 mm to (36.1, 68.6)
- moved J5 0.32 mm to (81.8, 60.5), turned to 0 degrees
Connections:
- net +10V renamed +10VSW
- net ALARM_SW renamed ALARM_SCL
- C13 pad 1: +3V3 -> Net-(C13-Pad1)
- C14 pad 1: +3V3 -> Net-(C13-Pad1)
- C30 pad 1: +5VSW -> Net-(C30-Pad1)
- C31 pad 1: +5VSW -> Net-(C30-Pad1)
- J5 pad 3: +3V3 -> Net-(C13-Pad1)
- R20 pad 2: EXP -> EXP_SDA
- U3 pad 26: EXP -> BEEPER
- U3 pad 33: BEEPER -> EXP_SDA
- U9 pad 5: +5VSW -> Net-(C30-Pad1)
Routing:
- net EXP_SDA: track 0.00 -> 49.0 mm, vias 0 -> 4
- net Net-(C13-Pad1): track 0.00 -> 37.2 mm, vias 0 -> 2
- net Net-(C30-Pad1): track 0.00 -> 21.0 mm, vias 0 -> 2
- net EXP: track 18.7 -> 0.00 mm, vias 2 -> 0
- net Net-(BZ1-Pad2): track 7.28 -> 20.5 mm, vias 1 -> 2
- net +10VSW: track 1.61 -> 13.0 mm, vias 0 -> 2
- net /Front Panel/R_LCD_MOSI: track 13.5 -> 2.98 mm
- net /Front Panel/R_BTN: track 7.77 -> 15.9 mm
- net /Front Panel/R_LCD_CLK: track 13.1 -> 5.31 mm, vias 0 -> 2
- net /Front Panel/R_BEEPER: track 10.5 -> 17.1 mm
- net /Front Panel/R_LCD_BL: track 11.4 -> 17.8 mm
- net /Front Panel/R_LCD_3.3V: track 21.6 -> 16.2 mm, vias 5 -> 7
- net N_PWR_LOSS: track 80.6 -> 75.7 mm
- net BEEPER: track 34.1 -> 29.3 mm, vias 4 -> 2
- net /Front Panel/R_LCD_DC: track 12.6 -> 8.67 mm, vias 0 -> 2
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Other:
- outline, holes or cut-outs redrawn
- board text added: "+10VSW"
- board text added: "GROVE I/O"
- board text added: "REV 0 / 2020-DEC-22"
- board text added: "◄◄◄ON"
- board text removed: "ALARM & EXP"
- board text removed: "REV 0 / 2020-DEC-21"
- board text removed: "REV 0 / 2020-DEC-21 FIAT LUX"
