File: hardware/uratt/uratt/uratt-power.sch (KiCad schematic (older format))
At the start: 68 parts, among them J6 Conn_01x02, J7 Conn_01x02, J8 Conn_01x02, SW4 SW_SPDT, U4 MCP73832-2-OT, U5 TPS2115A, U6 TPS61032PWP, U7 AP2112K-3.3, U8 AP2112K-3.3, U9 MP6513

Commit message: completed BOM, 3D STEP export
Parts:
- C17, C20: Digikey (none) -> 1276-1259-1-ND
- C18, C19: value .1uF -> 0.1uF; Digikey (none) -> 732-7939-1-ND
- C21, C22: Digikey (none) -> 587-2834-1-ND
- C23, C31: Digikey (none) -> 1276-1096-1-ND
- C24, C30: Digikey (none) -> 732-7939-1-ND
- C25, C26, C27: Digikey (none) -> 1276-1085-1-ND
- C28: Digikey (none) -> 478-6135-1-ND
- C29: Digikey (none) -> 1276-1942-1-ND; Field4 X75/X5R Ceramic -> X75/X5R Ceramic 25V
- D10: Digikey (none) -> BAT54SLT1GOSCT-ND
- D11, D7, D8, D9: Digikey (none) -> 732-4979-1-ND
- D12: Digikey (none) -> SM6T6V8A-E3/52GICT-ND
- F1: Digikey (none) -> 118-MF-NSHT075KX-2CT-ND
- GT1, H1, H2, H3, H4, TP1, TP2, TP3, TP4, TP5, TP6, TP7: Digikey (none) -> N/A
- J6, J7, J8: Digikey (none) -> 455-1704-ND
- JP1, JP2, JP3, JP4, JP5, JP6: Digikey (none) -> 2019-RK73Z1JTTDCT-ND
- L1: Digikey (none) -> 308-1937-1-ND; Field4 Sumida CDRH124-6R8 -> (none)
- R26: Digikey (none) -> 13-RT0603FRE072K05LCT-ND
- R27, R28, R31, R34, R41: Digikey (none) -> YAG2321CT-ND
- R29: Digikey (none) -> 13-RT0603FRE07270RLCT-ND
- R30, R35, R36, R37, R38, R42: Digikey (none) -> 13-RE0603FRE071KLCT-ND
- R32, R33, R39, R40: Digikey (none) -> TBD
- SW4: Digikey (none) -> 1948-1086-ND
- U4: value MCP73832-2-OT -> MCP73832T-2ACI/OT; Digikey (none) -> MCP73832T-2ACI/OTCT-ND
- U5: value TPS2115A -> TPS2115APWR; Digikey (none) -> 296-16940-1-ND
- U6: Digikey (none) -> 296-27007-5-ND
- U7, U8: value AP2112K-3.3 -> AP2112K-3.3TRG1; Digikey (none) -> AP2112K-3.3TRG1DICT-ND
- U9: value MP6513 -> MP6513GJ-Z; Digikey (none) -> 1589-1709-1-ND
