File: hardware/uratt/REV0/uratt/uratt.sch (KiCad schematic (older format))
At the start: 65 parts, among them J1 USB_B_Micro, J2 Micro_SD_Card, J3 Conn_01x10, J4 Conn_01x04, J5 Conn_01x04, Q1 MMBT3904, Q2 MMBT3904, SW1 SW_Push, SW2 SW_Push, U1 SN65220DBVR, U2 CP2102N-A02-GQFN24, U3 ESP32-WROOM-32E

Commit message: add REV0 ECO list.  start REV1 (copy of REV0)
Other:
- note added: "FRONT PANEL"
- note added: "POWER SUPPLY &\nMOTOR CONTROL"
Changed lines of the file:
@@
 Text Notes 14150 3400 0    50   ~ 0
 CONNECT J3 TO FRONT PANEL BOARD\n10POS 0.50MM FFC TOP/BOTTOM STYLE\n\nSAMTEC P/N  FJH-10-R-02.00-4\nhttp://suddendocs.samtec.com/catalog_english/fjh.pdf
+Text Notes 800  9750 0    118  ~ 0
+POWER SUPPLY &\nMOTOR CONTROL
+Text Notes 14950 1700 0    118  ~ 0
+FRONT PANEL
 $EndSCHEMATC
