File: hardware/uratt/REV1/uratt/uratt-frontpanel.sch (KiCad schematic (older format))
At the start: 28 parts, among them J9 Conn_01x10, Q3 DMP31D0U, Q4 2N7002, SW3 SW_Push

Commit message: work in progress on REV1 schematic/PCB
Parts:
- added R59: 470, Resistor_SMD:R_0603_1608Metric, symbol Device:R_Small_US
- added R61: 10K, Resistor_SMD:R_0603_1608Metric, symbol Device:R_Small_US
- BZ2: value Buzzer (ALT OPT) -> Buzzer (ALT)
- R51: value 220 -> 20
- R53: value 100 -> 10
Connections:
- net GND1: now also LCD1.11 (LED_K)
- net R_BTN: now also R61.2
- net R_LCD_3.3V: now also R61.1; no longer LCD1.11 (LED_K)
- net at BZ1.1 (-), BZ2.1 (-), R53.2: now also R59.1
- net at BZ1.2 (+), BZ2.2 (+), Q4.3 (D): now also R59.2
Other:
- moved on the sheet: C32, R43, SW3

Commit message: uratt REV1 work, remove front panel, place new parts, partial routing
Parts:
- removed BK1, BK2, BK3: BREAKAWAY, uratt:RATT_BITE, symbol uratt:BREAKAWAY
- removed BZ1: Buzzer, Buzzer_Beeper:Buzzer_CUI_CPT-9019S-SMT, symbol Device:Buzzer
- removed BZ2: Buzzer (ALT), Buzzer_Beeper:Buzzer_CUI_CPT-9019S-SMT, symbol Device:Buzzer
- removed C32, C34: 0.1uF, Capacitor_SMD:C_0603_1608Metric, symbol Device:C_Small
- removed C33: 1uF, Capacitor_SMD:C_0603_1608Metric, symbol Device:C_Small
- removed H5, H6, H7, H8: MountingHole, MountingHole:MountingHole_2.1mm, symbol Mechanical:MountingHole
- removed J9: Conn_01x10, Connector_FFC-FPC:TE_1-1734839-0_1x10-1MP_P0.5mm_Horizontal, symbol Connector_Generic:Conn_01x10
- removed LCD1: ER-TFT0.96-1, uratt:ER-TFT0.96-1, symbol uratt:ER-TFT0.96-1
- removed Q3: DMP31D0U, Package_TO_SOT_SMD:SOT-23, symbol Transistor_FET:BSS83P
- removed Q4: 2N7002, Package_TO_SOT_SMD:SOT-23, symbol Transistor_FET:2N7002
- removed R43, R46, R47, R48, R49, R50: 47, Resistor_SMD:R_0603_1608Metric, symbol Device:R_Small_US
- removed R44, R52: 1K, Resistor_SMD:R_0603_1608Metric, symbol Device:R_Small_US
- removed R45, R61: 10K, Resistor_SMD:R_0603_1608Metric, symbol Device:R_Small_US
- removed R51: 20, Resistor_SMD:R_0603_1608Metric, symbol Device:R_Small_US
- removed R53: 10, Resistor_SMD:R_0603_1608Metric, symbol Device:R_Small_US
- removed R59: 470, Resistor_SMD:R_0603_1608Metric, symbol Device:R_Small_US
- removed SW3: SW_Push, Button_Switch_SMD:SW_Push_1P1T_NO_CK_KSC6xxJ, symbol Switch:SW_Push
Connections:
- no-connect marks 2 -> 0
Other:
- note removed: "BACKLIGHT\nVF=3.2V IF=15mA\n"
- note removed: "GRAPHIC LCD"
